File: ai-hw-elec/ai-hw-elec.kicad_pcb (KiCad board)
At the start: 2 copper layers, 40.6 x 67.8 mm, 34 parts, among them J1 Conn_Progam_Stm, J2 Conn_01x02_power, SW1 Button_Push_TL3342, U1 ASM1117-3V3, U2 MP1584, U3 Stm32f103c8x, U4 LCD_ILI9341_2.2inch, Y1 Crystal-Mhz

Commit message: aa
Parts:
- added J3: Conn_01x04, phuong_kicad_lib:Header-4pin-2.54, F.Cu at (105.8, 74.3)
- added J4: Conn_01x04, phuong_kicad_lib:Header-4pin-2.54, F.Cu at (105.8, 59.1)
- added J5: Conn_01x04, phuong_kicad_lib:Header-4pin-2.54, F.Cu at (105.8, 90.2)
- added R10: R0805, phuong_kicad_lib:R_0805, F.Cu at (136.1, 78.6)
- added TH1: Thermistor_NTC, Resistor_THT:R_Axial_DIN0204_L3.6mm_D1.6mm_P1.90mm_Vertical, F.Cu at (138.4, 79.4)
Connections:
- U3 pad 10: (no net) -> /Stm32f103c8tx/adc_1
- U3 pad 12: (no net) -> /Stm32f103c8tx/uart2_tx
- U3 pad 13: (no net) -> /Stm32f103c8tx/uart2_rx
- U3 pad 30: (no net) -> /Stm32f103c8tx/uart1_tx
- U3 pad 31: (no net) -> /Stm32f103c8tx/uart1_rx
- U3 pad 42: (no net) -> /Stm32f103c8tx/i2c1_scl
- U3 pad 43: (no net) -> /Stm32f103c8tx/i2c1_sda
Routing:
- net 3V3: track 108.5 -> 160.2 mm
- net /Stm32f103c8tx/i2c1_scl: track 0.00 -> 44.0 mm, vias 0 -> 1
- net /Stm32f103c8tx/i2c1_sda: track 0.00 -> 43.7 mm, vias 0 -> 1
- net /Stm32f103c8tx/uart2_tx: track 0.00 -> 35.5 mm, vias 0 -> 1
- net /Stm32f103c8tx/uart2_rx: track 0.00 -> 35.5 mm, vias 0 -> 1
- net /Stm32f103c8tx/uart1_tx: track 0.00 -> 29.7 mm, vias 0 -> 1
- net /Stm32f103c8tx/uart1_rx: track 0.00 -> 28.3 mm, vias 0 -> 2
- net /Stm32f103c8tx/adc_1: track 0.00 -> 25.7 mm, vias 0 -> 1
- net GND: track 14.7 -> 15.6 mm, vias 6 -> 9
Other:
- board size 40.6 x 67.8 mm -> 48.3 x 67.8 mm
- board text added: "12v"
- board text added: "3v3"
- board text added: "gnd"
- board text added: "res"
- board text added: "rx1"
- board text added: "rx2"
- board text added: "scl1"
- board text added: "sda1"
- board text added: "swclk"
- board text added: "swdio"
- board text added: "tx1"
- board text added: "tx2"

Commit message: add
Parts:
- removed TH1: Thermistor_NTC, Resistor_THT:R_Axial_DIN0204_L3.6mm_D1.6mm_P1.90mm_Vertical
- added C11: 104, ph_kicad_lib:C_0805_HandSoldering, F.Cu at (124.9, 87.8)
- added C12: 104, ph_kicad_lib:C_0805_HandSoldering, F.Cu at (106.8, 87.8)
- added D2: D_TVS, ph_kicad_lib:DO-214AC(SMA), F.Cu at (130.4, 79.8)
- added D3: D_TVS, ph_kicad_lib:DO-214AC(SMA), F.Cu at (112.2, 79.8)
- added J6: 5v lock, phuong_kicad_lib:Header-2pin-2.54-white, F.Cu at (117.1, 105.4)
- added J7: 3v3 lock, phuong_kicad_lib:Header-2pin-2.54-white, F.Cu at (106.4, 111.0)
- added J8: Conn_01x02_power, phuong_kicad_lib:Header-2pin-2.54-white, F.Cu at (144.3, 103.1)
- added J9: Conn_01x02_power, phuong_kicad_lib:Header-2pin-2.54-white, F.Cu at (144.3, 96.3)
- added Q1: C1815_SOT23, ph_kicad_lib:SOT-23, F.Cu at (131.2, 95.9)
- added Q2: C1815_SOT23, ph_kicad_lib:SOT-23, F.Cu at (113.0, 95.5)
- added R11: 2.2k, ph_kicad_lib:R_0805_HandSoldering, F.Cu at (130.4, 83.3)
- added R12: 10K, ph_kicad_lib:R_0805_HandSoldering, F.Cu at (125.8, 84.0)
- added R13: 10k, ph_kicad_lib:R_0805_HandSoldering, F.Cu at (126.3, 91.5)
- added R14: 10k, ph_kicad_lib:R_0805_HandSoldering, F.Cu at (123.5, 91.6)
- added R15: 4k7, ph_kicad_lib:R_0805_HandSoldering, F.Cu at (136.2, 90.5)
- added R16: 2.2k, ph_kicad_lib:R_0805_HandSoldering, F.Cu at (136.2, 95.3)
- added R17: 10k, ph_kicad_lib:R_0805_HandSoldering, F.Cu at (136.1, 92.9)
- added R18: 10K, ph_kicad_lib:R_0805_HandSoldering, F.Cu at (117.9, 84.6)
- added R19: 2.2k, ph_kicad_lib:R_0805_HandSoldering, F.Cu at (112.1, 83.0)
- added R20: 10K, ph_kicad_lib:R_0805_HandSoldering, F.Cu at (106.1, 84.0)
- added R21: 10k, ph_kicad_lib:R_0805_HandSoldering, F.Cu at (107.9, 91.4)
- added R22: 10k, ph_kicad_lib:R_0805_HandSoldering, F.Cu at (105.7, 91.5)
- added R23: 4k7, ph_kicad_lib:R_0805_HandSoldering, F.Cu at (118.0, 92.3)
- added R24: 2.2k, ph_kicad_lib:R_0805_HandSoldering, F.Cu at (117.9, 97.2)
- added R25: 10k, ph_kicad_lib:R_0805_HandSoldering, F.Cu at (118.0, 94.7)
- added U5: MAX485_SMD, ph_kicad_lib:SOIC-8_3.9x4.9mm_Pitch1.27mm, F.Cu at (130.5, 89.5)
- added U6: MAX485_SMD, ph_kicad_lib:SOIC-8_3.9x4.9mm_Pitch1.27mm, F.Cu at (112.1, 89.5)
- J2: value Conn_01x02_power -> RS485_uart1
- J3: value Conn_01x04 -> RS485_uart2; footprint phuong_kicad_lib:Header-4pin-2.54 -> phuong_kicad_lib:Header-2pin-2.54-white
- J4: value Conn_01x04 -> Conn_01x02_power; footprint phuong_kicad_lib:Header-4pin-2.54 -> phuong_kicad_lib:Header-2pin-2.54-white
- J5: value Conn_01x04 -> I2C_Port
- R10: value R0805 -> 10K; footprint phuong_kicad_lib:R_0805 -> ph_kicad_lib:R_0805_HandSoldering
- moved J2 71.6 mm to (105.6, 57.8), turned to 0 degrees
- moved J4 69.9 mm to (144.5, 117.3), turned to 90 degrees
- moved R5 35.1 mm to (106.4, 118.1), turned to 0 degrees
- moved Led1 34.8 mm to (106.4, 120.4), turned to 0 degrees
- moved C2 27.2 mm to (112.5, 112.8), turned to 0 degrees
- moved CP2 27.0 mm to (112.5, 109.7), turned to 0 degrees
- moved U1 26.8 mm to (114.6, 118.1), turned to 180 degrees
- moved J5 19.2 mm to (105.1, 71.0)
- moved C1 15.2 mm to (118.6, 112.8), turned to 0 degrees
- moved J3 10.3 mm to (105.7, 64.0)
- moved R6 8.38 mm to (132.1, 116.6)
- moved R7 8.38 mm to (132.1, 114.0)
- moved U2 8.38 mm to (134.4, 109.5)
- moved C3 8.38 mm to (141.5, 107.7)
- moved C4 8.38 mm to (127.5, 116.6)
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Connections:
- C1 pad 1: 5v -> Net-(C1-Pad1)
- C2 pad 1: 3V3 -> Net-(C2-Pad1)
- CP2 pad 1: 3V3 -> Net-(C2-Pad1)
- J2 pad 1: 12v -> /rs485uart1/A
- J2 pad 2: GND -> /rs485uart1/B
- J3 pad 1: 3V3 -> /rs485uart2/A
- J3 pad 2: /Stm32f103c8tx/uart1_rx -> /rs485uart2/B
- J4 pad 1: 3V3 -> 12v
- J4 pad 2: /Stm32f103c8tx/uart2_rx -> GND
- L2 pad 2: GND -> Net-(L2-Pad2)
- R10 pad 1: 3V3 -> 5v
- R10 pad 2: /Stm32f103c8tx/adc_1 -> /rs485uart1/A
- U1 pad 2: 3V3 -> Net-(C2-Pad1)
- U1 pad 3: 5v -> Net-(C1-Pad1)
- U1 pad 4: 3V3 -> Net-(C2-Pad1)
- U3 pad 1: (no net) -> Net-(U3-Pad1)
- U3 pad 11: (no net) -> Net-(U3-Pad11)
- U3 pad 12: /Stm32f103c8tx/uart2_tx -> /rs485uart2/RS485-TX
- U3 pad 13: /Stm32f103c8tx/uart2_rx -> /rs485uart2/RS485-RX
- U3 pad 18: (no net) -> Net-(U3-Pad18)
- U3 pad 19: (no net) -> Net-(U3-Pad19)
- U3 pad 2: (no net) -> Net-(U3-Pad2)
- U3 pad 25: (no net) -> Net-(U3-Pad25)
- U3 pad 26: (no net) -> Net-(U3-Pad26)
- U3 pad 27: (no net) -> Net-(U3-Pad27)
- U3 pad 28: (no net) -> Net-(U3-Pad28)
- U3 pad 29: (no net) -> Net-(U3-Pad29)
- U3 pad 3: (no net) -> Net-(U3-Pad3)
- U3 pad 30: /Stm32f103c8tx/uart1_tx -> /rs485uart1/RS485-TX
- U3 pad 31: /Stm32f103c8tx/uart1_rx -> /rs485uart1/RS485-RX
- U3 pad 32: (no net) -> Net-(U3-Pad32)
- U3 pad 33: (no net) -> Net-(U3-Pad33)
- U3 pad 38: (no net) -> Net-(U3-Pad38)
- U3 pad 39: (no net) -> Net-(U3-Pad39)
- U3 pad 4: (no net) -> Net-(U3-Pad4)
- U3 pad 40: (no net) -> Net-(U3-Pad40)
- U3 pad 41: (no net) -> Net-(U3-Pad41)
- U3 pad 45: (no net) -> Net-(U3-Pad45)
- U3 pad 46: (no net) -> Net-(U3-Pad46)
- U3 pad 9: 3V3 -> Net-(L2-Pad2)
- U4 pad 10: (no net) -> Net-(U4-Pad10)
- U4 pad 11: (no net) -> Net-(U4-Pad11)
- U4 pad 12: (no net) -> Net-(U4-Pad12)
- U4 pad 13: (no net) -> Net-(U4-Pad13)
- U4 pad 14: (no net) -> Net-(U4-Pad14)
Routing:
- net 5v: track 29.6 -> 122.5 mm
- net /rs485uart1/A: track 0.00 -> 51.6 mm
- net /rs485uart1/B: track 0.00 -> 46.7 mm
- net /Stm32f103c8tx/i2c1_scl: track 44.0 -> 0.00 mm, vias 1 -> 0
- net /Stm32f103c8tx/i2c1_sda: track 43.7 -> 0.00 mm, vias 1 -> 0
- net /Stm32f103c8tx/uart2_tx: track 35.5 -> 0.00 mm, vias 1 -> 0
- net /Stm32f103c8tx/uart2_rx: track 35.5 -> 0.00 mm, vias 1 -> 0
- net /rs485uart2/A: track 0.00 -> 33.1 mm
- net /rs485uart2/B: track 0.00 -> 31.2 mm
- net /Stm32f103c8tx/uart1_tx: track 29.7 -> 0.00 mm, vias 1 -> 0
- net /Stm32f103c8tx/uart1_rx: track 28.3 -> 0.00 mm, vias 2 -> 0
- net /Stm32f103c8tx/adc_1: track 25.7 -> 0.00 mm, vias 1 -> 0
- net 3V3: track 160.2 -> 138.5 mm, vias 5 -> 4
- net Net-(C2-Pad1): track 0.00 -> 20.3 mm
- net Net-(Q1-Pad3): track 0.00 -> 13.6 mm
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Other:
- board text removed: "12v"
- board text removed: "3v3"
- board text removed: "rx1"
- board text removed: "rx2"
- board text removed: "scl1"
- board text removed: "sda1"
- board text removed: "tx1"
- board text removed: "tx2"

Commit message: add
Parts:
- moved R9 1.30 mm to (135.1, 74.4)
- moved C8 1.25 mm to (137.4, 74.5)
Routing:
- net /rs485uart2/RS485-TX: track 3.13 -> 59.3 mm, vias 1 -> 3
- net /rs485uart2/RS485-RX: track 3.11 -> 53.9 mm, vias 0 -> 2
- net /rs485uart1/RS485-TX: track 2.25 -> 49.4 mm, vias 1 -> 2
- net /rs485uart1/RS485-RX: track 5.20 -> 47.1 mm, vias 1 -> 2
- net /Stm32f103c8tx/i2c1_scl: track 0.00 -> 32.5 mm, vias 0 -> 1
- net 3V3: track 138.5 -> 168.9 mm
- net /Stm32f103c8tx/i2c1_sda: track 0.00 -> 30.1 mm, vias 0 -> 1
- net Net-(L2-Pad2): track 0.00 -> 14.6 mm
- net GND: track 26.2 -> 30.9 mm, vias 12 -> 13
- net /LCD-MISO: track 13.6 -> 16.3 mm
- net Net-(R9-Pad1): track 3.02 -> 3.79 mm
